File: PCB/specter/specter.kicad_pcb (KiCad board)
At the start: 4 copper layers, 65 x 67 mm, 94 parts, among them J1 USB_C_Receptacle_USB2.0_16P, J2 Micro_SD_Card_Det2, J22 SM04B-SRSS-TB_LF__SN_, J23 Conn_01x01, J24 SM04B-SRSS-TB_LF__SN_, J25 SM04B-SRSS-TB_LF__SN_, J26 SM04B-SRSS-TB_LF__SN_, J27 SM06B-SRSS-TB_LF__SN_, J28 SM06B-SRSS-TB_LF__SN_, J29 SM06B-SRSS-TB_LF__SN_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

Commit message: finalised routing on PCB
Parts:
- removed J7: Conn_01x03, Jumper:SolderJumper-3_P1.3mm_Open_RoundedPad1.0x1.5mm_NumberLabels
- TP35: moved to F.Cu
- moved JP1 3.89 mm to (115.2, 112.2), turned to 90 degrees
- moved JP6 1.80 mm to (123.6, 126.2), turned to 90 degrees
- moved TP35 1.66 mm to (155.7, 84.5)
Routing:
- net /GPIO3: track 0.00 -> 48.8 mm
- net /GPIO2: track 0.00 -> 46.5 mm
- net /PWR_BUT: track 10.2 -> 35.5 mm, vias 0 -> 2
- net /SD_PWR: track 0.00 -> 23.4 mm, vias 0 -> 3
- net /GPIO10: track 8.84 -> 22.2 mm
- net /SD_PWR_ON: track 0.00 -> 11.1 mm, vias 0 -> 2
- net /nRPIBOOT: track 0.00 -> 5.66 mm
- net /TX_TELEM: track 26.6 -> 29.8 mm
- net /CE0: track 27.0 -> 24.2 mm
- net /PMIC_ENABLE: track 15.4 -> 13.9 mm
- net Net-(U1-3V3OUT): track 18.3 -> 17.2 mm

Commit message: small PCB updates
Routing:
- net /+5v: track 8.55 -> 12.9 mm, vias 3 -> 32
- net /nPWR_LED: track 21.2 -> 22.5 mm, vias 0 -> 2
- net GND: vias 0 -> 34
- added copper zone on B.Cu, net /+5v
- added copper zone on F.Cu, net /+5v
- added copper zone on F.Cu, net GND
- added copper zone on In1.Cu, net GND

Commit message: added power planes
Routing:
- net /PCIE_PWR_EN: track 2.20 -> 57.5 mm, vias 0 -> 2
- net /+5v: track 12.9 -> 64.1 mm, vias 32 -> 42
- net /+3.3v: track 0.00 -> 40.7 mm, vias 0 -> 5
- net /LED_nACT: track 9.18 -> 31.4 mm
- net /+1.8v: track 0.00 -> 11.8 mm, vias 0 -> 3
- net /VBUS: track 27.5 -> 31.3 mm
- added copper zone on In2.Cu, net /+5v
- added copper zone on B.Cu, net GND
