File: PCB/specter/specter.kicad_pcb (KiCad board)
At the start: 4 copper layers, 65 x 67 mm, 93 parts, among them J1 USB_C_Receptacle_USB2.0_16P, J2 Micro_SD_Card_Det2, J22 SM04B-SRSS-TB_LF__SN_, J23 Conn_01x01, J24 SM04B-SRSS-TB_LF__SN_, J25 SM04B-SRSS-TB_LF__SN_, J26 SM04B-SRSS-TB_LF__SN_, J27 SM06B-SRSS-TB_LF__SN_, J28 SM06B-SRSS-TB_LF__SN_, J29 SM06B-SRSS-TB_LF__SN_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

Commit message: added last minute changes
Routing:
- net /VBUS: track 83.3 -> 129.7 mm
- net GND: track 10.6 -> 52.4 mm, vias 49 -> 70
- net /GPIO_VREF: track 43.0 -> 65.5 mm
- net /+5v: vias 46 -> 30
- removed copper zone on B.Cu, net /+5v

Commit message: refined PCB
Routing:
- net GND: track 52.4 -> 29.7 mm
- net /+5v: track 146.6 -> 156.0 mm
- net /PCIE_RX_P: track 28.9 -> 37.4 mm
- net /PCIE_RX_N: track 34.5 -> 37.5 mm
- net /PCIE_TX_P: track 32.3 -> 34.6 mm
- net /PCIE_TX_N: track 33.0 -> 34.6 mm
Other:
- board text added: "26 | 19 | 13 | 6 | 5 | 4"
- board text added: "Main"
- board text added: "Real Small"
- board text added: "Small"
- board text added: "Sub-head"

Commit message: finishing touches
Parts:
- added G***: LOGO, Logo:ASRS_logo_20x20, F.Cu at (151.0, 126.8)
- added G***: LOGO, Logo:barcode_10m, F.Cu at (124.0, 72.2)
- added G***: LOGO, Logo:flag_lv_inv_10mm, F.Cu at (115.6, 83.3)
- added G***: LOGO, Logo:asrs_pilot_qr_7x7, B.Cu at (157.5, 124.7)
Routing:
- net /DPHY0_D2_N: track 17.3 -> 17.8 mm
- net /DPHY0_D2_P: track 17.3 -> 17.8 mm
- net GND: vias 70 -> 86
- net /+5v: vias 30 -> 20
Other:
- board text added: "+5V"
- board text added: "+5V | 11 | 09 | 10 | 8 | GND"
- board text added: "+5V | TX | RX |GND"
- board text added: "21 | 20 | 16 | 12 | 7 | 25"
- board text added: "Cam/Disp 0"
- board text added: "Cam/Disp 1"
- board text added: "Desined in LV."
- board text added: "EEPROM-nWP"
- board text added: "GND"
- board text added: "Jump two for DPHY1"
- board text added: "PMIC_EN"
- board text added: "PWR_SW"
- board text added: "PiLOT Dev. Board 1.0"
- board text added: "Sync_out"
- board text added: "This is the pilot. You are the visionary. We built this board as fellow makers so you can push the limits of what's possible. Now, take flight and build something extraordinary."
- board text added: "UART1"
- board text added: "UART2"
- board text added: "USB OTG"
- board text added: "Your build. Your imagination. Your rules."
- board text added: "nRPIBOOT"
- board text added: "Šis ir pilots. Jūs esat vizionārs. Mēs veidojām šo dēli kā citi veidotāji lai jūs varētu pārkāpt iespējamās robežas. Tagad lidojiet un izveidojiet kaut ko neparastu."

Commit message: added 3D models
Parts:
- removed the G*** at (115.6, 83.3)
Other:
- board text removed: "Desined in LV."
- board text removed: "Main"
- board text removed: "Real Small"
- board text removed: "Small"
- board text removed: "Sub-head"

Commit message: final PCB changes
Parts:
- removed R15, R16: 0R, Resistor_SMD:R_0805_2012Metric_Pad1.20x1.40mm_HandSolder
- removed R4, R6: 0, Resistor_SMD:R_0805_2012Metric_Pad1.20x1.40mm_HandSolder
- added J6: DF40C-100DS-0.4V_51_, DF40C-100DS-0:HIROSE_DF40C-100DS-0.4V_51_, F.Cu at (114.5, 98.7)
- added J9: DF40C-100DS-0.4V_51_, DF40C-100DS-0:HIROSE_DF40C-100DS-0.4V_51_, F.Cu at (148.5, 98.7)
Connections:
- C4 pad 2: Net-(C4-Pad2) -> /VBUS
- C5 pad 1: Net-(C4-Pad2) -> /VBUS
- C6 pad 2: Net-(C6-Pad2) -> /VBUS
- C7 pad 1: Net-(C6-Pad2) -> /VBUS
- Module1 pad 78: /GPIO_VREF -> /+3.3v
- R13 pad 2: /GPIO_VREF -> /+3.3v
- R14 pad 1: /GPIO_VREF -> /+3.3v
- R5 pad 2: Net-(C4-Pad2) -> /VBUS
- R7 pad 2: Net-(C6-Pad2) -> /VBUS
Routing:
- net /GPIO_VREF: track 65.5 -> 0.00 mm, vias 4 -> 0
- net /VBUS: track 129.7 -> 164.3 mm, vias 6 -> 10
- net /+3.3v: track 150.8 -> 184.4 mm, vias 10 -> 12
- net Net-(C4-Pad2): track 21.9 -> 0.00 mm, vias 4 -> 0
- net /+1.8v: track 21.5 -> 0.40 mm, vias 2 -> 0
- net Net-(C6-Pad2): track 7.49 -> 0.00 mm
Other:
- board text removed: "Cam/Disp 0"
- board text removed: "Cam/Disp 1"
