File: PCB/specter/_autosave-specter.kicad_pcb (KiCad board)
At the start: 4 copper layers, 65 x 67 mm, 93 parts, among them J1 USB_C_Receptacle_USB2.0_16P, J2 Micro_SD_Card_Det2, J22 SM04B-SRSS-TB_LF__SN_, J23 Conn_01x01, J24 SM04B-SRSS-TB_LF__SN_, J25 SM04B-SRSS-TB_LF__SN_, J26 SM04B-SRSS-TB_LF__SN_, J27 SM06B-SRSS-TB_LF__SN_, J28 SM06B-SRSS-TB_LF__SN_, J29 SM06B-SRSS-TB_LF__SN_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

Commit message: finished PCB first round
Routing:
- net /VBUS: track 83.3 -> 129.7 mm
- net GND: track 10.6 -> 52.4 mm, vias 49 -> 53
- net /GPIO_VREF: track 43.0 -> 63.5 mm
Changed lines of the file:
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@@
 	)
 	(segment
+		(start 102.125 116.473)
+		(end 103.327 116.473)
+		(width 0.35)
+		(layer "F.Cu")
+		(net 1)
+	)
+	(segment
+		(start 114.1565 102.925)
+		(end 114.5565 103.325)
+		(width 0.2)
+		(layer "F.Cu")
+		(net 1)
+	)
+	(segment
 		(start 146.96 90.125)
 		(end 147.325 90.125)
@@
 	)
 	(segment
+		(start 109.7 120.6)
+		(end 109.5 120.4)
+		(width 0.35)
+		(layer "F.Cu")
+		(net 1)
+	)
+	(segment
+		(start 112.96 102.925)
+		(end 114.1565 102.925)
+		(width 0.2)
+		(layer "F.Cu")
+		(net 1)
+	)
+	(segment
 		(start 147.599 92.251)
 		(end 147.325 92.525)
@@
 	)
 	(segment
+		(start 109.7 122.4)
+		(end 109.7 120.6)
+		(width 0.35)
+		(layer "F.Cu")
+		(net 1)
+	)
+	(segment
+		(start 109.3 124.9)
+		(end 110.1 124.9)
+		(width 0.35)
+		(layer "F.Cu")
+		(net 1)
+	)
+	(segment
+		(start 103.327 116.473)
+		(end 104.627 115.173)
+		(width 0.35)
+		(layer "F.Cu")
+		(net 1)
+	)
+	(segment
 		(start 133 113.75)
 		(end 132.25 113.75)
@@
 	)
 	(segment
+		(start 104.627 115.173)
+		(end 106 115.173)
+		(width 0.35)
+		(layer "F.Cu")
+		(net 1)
+	)
+	(segment
+		(start 114.5565 103.325)
+		(end 116.04 103.325)
+		(width 0.2)
+		(layer "F.Cu")
+		(net 1)
+	)
+	(segment
+		(start 110.1 124.9)
+		(end 110.2 124.8)
+		(width 0.35)
+		(layer "F.Cu")
+		(net 1)
+	)
+	(segment
 		(start 132.25 113.75)
 		(end 131.7515 113.2515)
@@
 	)
 	(via
+		(at 123.6 126.8)
+		(size 0.45)
+		(drill 0.2)
+		(layers "F.Cu" "B.Cu")
+		(net 1)
+	)
+	(via
 		(at 157.5 70.5)
 		(size 0.45)
@@
 	)
 	(via
+		(at 110.2 124.8)
+		(size 0.45)
+		(drill 0.2)
+		(layers "F.Cu" "B.Cu")
+		(free yes)
+		(net 1)
+	)
+	(via
 		(at 113.1 125.25)
 		(size 0.45)
@@
 	)
 	(via
+		(at 115.1 92)
+		(size 0.45)
+		(drill 0.2)
+		(layers "F.Cu" "B.Cu")
+		(free yes)
+		(net 1)
+	)
+	(via
 		(at 134.2 77.3)
 		(size 0.45)
@@
 	)
 	(via
+		(at 109.7 122.4)
+		(size 0.45)
+		(drill 0.2)
+		(layers "F.Cu" "B.Cu")
+		(free yes)
+		(net 1)
+	)
+	(via
 		(at 155 125.5)
 		(size 0.45)
@@
 	)
 	(segment
+		(start 102.925 122.9)
+		(end 100.8 120.775)
+		(width 0.2)
+		(layer "B.Cu")
+		(net 1)
+	)
+	(segment
 		(start 156.3 112.95)
 		(end 155.9 112.55)
@@
 	)
 	(segment
+		(start 112.965 92)
+		(end 115.1 92)
+		(width 0.35)
+		(layer "B.Cu")
+		(net 1)
+	)
+	(segment
 		(start 155.9 114.65)
 		(end 155.9 112.55)
@@
 	)
 	(segment
+		(start 100.8 120.775)
+		(end 100.8 94.8)
+		(width 0.2)
+		(layer "B.Cu")
+		(net 1)
+	)
+	(segment
 		(start 153.27 75.9)
 		(end 153.65 75.52)
@@
 	)
 	(segment
+		(start 115.590114 92.8)
+		(end 110.2 92.8)
+		(width 0.35)
+		(layer "B.Cu")
+		(net 8)
+	)
+	(segment
+		(start 127.7 101.4)
+		(end 124.190114 101.4)
+		(width 0.35)
+		(layer "B.Cu")
+		(net 8)
+	)
+	(segment
 		(start 157.7 119.7)
 		(end 159.2875 118.1125)
@@
 	)
 	(segment
+		(start 110.2 92.8)
+		(end 106 88.6)
+		(width 0.35)
+		(layer "B.Cu")
+		(net 8)
+	)
+	(segment
 		(start 154.1625 116.5)
 		(end 155 116.5)
@@
 	)
 	(segment
+		(start 106 88.6)
+		(end 106 86.575)
+		(width 0.35)
+		(layer "B.Cu")
+		(net 8)
+	)
+	(segment
 		(start 156.363738 119.7)
 		(end 157.7 119.7)
@@
 	)
 	(segment
+		(start 124.190114 101.4)
+		(end 115.590114 92.8)
+		(width 0.35)
+		(layer "B.Cu")
+		(net 8)
+	)
+	(segment
+		(start 123.7 114.3)
+		(end 130.1 107.9)
+		(width 0.35)
+		(layer "B.Cu")
+		(net 8)
+	)
+	(segment
 		(start 109.994738 84.275)
 		(end 109.3 84.969738)
@@
 	)
 	(segment
+		(start 122.8 114.3)
+		(end 123.7 114.3)
+		(width 0.35)
+		(layer "B.Cu")
+		(net 8)
+	)
+	(segment
 		(start 159.2875 118.1125)
 		(end 161.4 118.1125)
@@
 	)
 	(segment
+		(start 130.1 103.8)
+		(end 127.7 101.4)
+		(width 0.35)
+		(layer "B.Cu")
+		(net 8)
+	)
+	(segment
 		(start 150.5 112)
 		(end 150 112)
@@
 	)
 	(segment
+		(start 130.1 107.9)
+		(end 130.1 103.8)
+		(width 0.35)
+		(layer "B.Cu")
+		(net 8)
+	)
+	(segment
 		(start 110.8 84.275)
 		(end 109.994738 84.275)
@@
 		(net 159)
 	)
+	(segment
+		(start 118.423545 104)
+		(end 121.1 104)
+		(width 0.2)
+		(layer "In2.Cu")
+		(net 159)
+	)
+	(segment
+		(start 108.3 114.1)
+		(end 108.3 108)
+		(width 0.2)
+		(layer "In2.Cu")
+		(net 159)
+	)
+	(segment
+		(start 118.1 104.323545)
+		(end 118.423545 104)
+		(width 0.2)
+		(layer "In2.Cu")
+		(net 159)
+	)
+	(segment
+		(start 108.3 108)
+		(end 111.976455 104.323545)
+		(width 0.2)
+		(layer "In2.Cu")
+		(net 159)
+	)
+	(segment
+		(start 111.976455 104.323545)
+		(end 118.1 104.323545)
+		(width 0.2)
+		(layer "In2.Cu")
+		(net 159)
+	)
