File: PCB/specter/specter.kicad_sch (KiCad schematic)
At the start: 73 parts, among them J1 USB_C_Receptacle_USB2.0_16P, J2 Micro_SD_Card_Det2, J3 THD-02-R, J4 Conn_01x22_Socket, J5 Conn_01x22_Socket, J7 Conn_01x03, J8 Conn_01x04, SW1 SW_Omron_B3FS, U1 FT232RL, U2 FT232RL, U3 RT9742GGJ5, U4 MagJack-A70-112-331N126, U5 TPD4EUSB30, U6 TPD4EUSB30, U7 74LVC1G07_copy, U8 AP2553W6

Commit message: pre-check schematic layout
Parts:
- removed J8: Conn_01x04, symbol Connector_Generic:Conn_01x04
- removed SW1: SW_Omron_B3FS, symbol Switch:SW_Omron_B3FS
- added C15: 22uF, symbol Device:C_Small
- added C16: 10uF, symbol Device:C_Small
- added J10: Conn_01x01, TestPoint:TestPoint_Loop_D2.54mm_Drill1.5mm_Beaded, symbol Connector_Generic:Conn_01x01
- added J11, J12, J13, J14, J15, J16, J17, J18, J19, J20, J21: Conn_01x01, symbol Connector_Generic:Conn_01x01
- added J22, J24, J25, J26: SM04B-SRSS-TB_LF__SN_, SM04B-SRSS-TB_LF__SN_:JST_SM04B-SRSS-TB_LF__SN_, symbol SM04B-SRSS-TB_LF__SN_:SM04B-SRSS-TB_LF__SN_
- added J23, J8: Conn_01x01, TestPoint:TestPoint_THTPad_4.0x4.0mm_Drill2.0mm, symbol Connector_Generic:Conn_01x01
- added J27, J28, J29, J30: SM06B-SRSS-TB_LF__SN_, JST_SM06B-SRSS-TB_LF__SN_, symbol SM06B-SRSS-TB_LF__SN_:SM06B-SRSS-TB_LF__SN_
- added J6, J9: Conn_01x01, TestPoint:TestPoint_THTPad_3.0x3.0mm_Drill1.5mm, symbol Connector_Generic:Conn_01x01
- added R20: 420R, symbol Device:R_Small
- added R21: 140R, symbol Device:R_Small
- added S1: SKQGAFE010, SKQGAFE010:SW_SKQGAFE010, symbol SKQGAFE010:SKQGAFE010
- added TP10, TP11, TP12, TP13, TP14, TP15, TP16, TP17, TP18, TP19, TP20, TP21, TP22, TP23, TP24, TP25, TP26, TP27, TP28, TP29, TP30, TP31, TP32, TP33, TP34, TP35, TP36, TP7, TP8, TP9: TestPoint, TestPoint:TestPoint_Pad_D1.0mm, symbol Connector:TestPoint
- added U9: MIC29752WT, Package_TO_SOT_THT:TO-247-5_Vertical, symbol Regulator_Linear:MIC29752WT
- C3, C9: footprint (none) -> Capacitor_SMD:C_0603_1608Metric_Pad1.08x0.95mm_HandSolder
- D1, D2, D3, D4, D5, D6: footprint (none) -> LED_SMD:LED_0603_1608Metric_Pad1.05x0.95mm_HandSolder
- D7: value LED -> LED RED
- J1: footprint (none) -> CM5IO:EDAC 690-019-298-412
- J5: footprint (none) -> CM5IO:Hirose_FH12-22S-0.5SH_1x22-1MP_P0.50mm_Horizontal
- J7: footprint (none) -> Jumper:SolderJumper-3_P1.3mm_Open_RoundedPad1.0x1.5mm_NumberLabels
- R2, R3, R6, R7, R8, R9: footprint (none) -> Resistor_SMD:R_0603_1608Metric_Pad0.98x0.95mm_HandSolder
Connections:
- net SCL1 is gone; now on net GPIO2: J5.20 (Pin_20)
- net SDA0 is gone; now on net GPIO3: J4.21 (Pin_21), JP8.2 (B), Module1.82 (SDA0), R13.1
- net +3.3v: now also J10.1 (Pin_1), J11.1 (Pin_1), J12.1 (Pin_1), TP33.1, TP36.1
- net +5v: now also C16.1, J13.1 (Pin_1), J14.1 (Pin_1), J15.1 (Pin_1), J22.1, J24.1, J25.1, J26.1, J27.1, J6.1 (Pin_1), R20.1, TP34.1, TP35.1, U9.4 (VOUT)
- net GND: now also J7.2 (Pin_2), Module2.107 (GND), Module2.108 (GND), Module2.113 (GND), Module2.114 (GND), Module2.119 (GND), Module2.120 (GND), Module2.125 (GND), Module2.126 (GND), Module2.131 (GND), Module2.132 (GND), Module2.137 (GND), Module2.138 (GND), Module2.144 (GND), Module2.150 (GND), Module2.155 (GND), Module2.156 (GND), Module2.161 (GND), Module2.162 (GND), Module2.167 (GND), Module2.168 (GND), Module2.173 (GND), Module2.174 (GND), Module2.179 (GND), Module2.180 (GND), Module2.185 (GND), Module2.186 (GND), Module2.191 (GND), Module2.192 (GND), Module2.197 (GND), Module2.198 (GND), C15.2, C16.2, J16.1 (Pin_1), J17.1 (Pin_1), J18.1 (Pin_1), J19.1 (Pin_1), J20.1 (Pin_1), J21.1 (Pin_1), J22.4, J22.S1 (SHIELD), J22.S2 (SHIELD), J24.4, J24.S1 (SHIELD), J24.S2 (SHIELD), J25.4, J25.S1 (SHIELD), J25.S2 (SHIELD), J26.4, J26.S1 (SHIELD), J26.S2 (SHIELD), J27.6, J27.S1 (SHIELD), J27.S2 (SHIELD), J28.S1 (SHIELD), J28.S2 (SHIELD), J29.S1 (SHIELD), J29.S2 (SHIELD), J30.S1 (SHIELD), J30.S2 (SHIELD), J8.1 (Pin_1), J9.1 (Pin_1), R21.2, S1.3, S1.4, U9.3 (GND)
- net GPIO10: now also J27.4, TP14.1, TP28.1
- net GPIO11: now also J27.2, TP12.1, TP19.1
- net GPIO12: now also J28.5, TP24.1
- net GPIO13: now also J28.6, TP9.1
- net GPIO14: now also J22.2
- net GPIO15: now also J22.3
- net GPIO16: now also J29.1, TP23.1
- net GPIO17: now also J29.2, TP17.1
- net GPIO18: now also J29.3, TP27.1
- net GPIO19: now also J29.4, TP8.1
- net GPIO2: now also J26.3
- net GPIO20: now also J29.5, TP22.1
- net GPIO21: now also J29.6, TP21.1
- net GPIO22: now also J30.1, TP15.1
- net GPIO23: now also J30.2, TP26.1
- net GPIO24: now also J30.3, TP25.1
- net GPIO25: now also J30.4, TP31.1
- net GPIO26: now also J30.5, TP7.1
- net GPIO27: now also J30.6, TP16.1
- net GPIO3: now also J26.2
- net GPIO4: now also J28.1, TP18.1
- net GPIO5: now also J28.2, TP11.1
- net GPIO6: now also J28.3, TP10.1
- net GPIO7: now also J28.4, TP29.1
- net GPIO9: now also J27.3, TP13.1, TP20.1
- net PWR_BUT: now also S1.1, S1.2, TP32.1
- net GPIO8 renamed CE0
- net CE0: now also J27.5, TP30.1
- net RX_CRSF renamed RX2
- net RX2: now also J25.3
- net RX_TELEM renamed RX1
- net RX1: now also J24.3
- net TX_CRSF renamed TX2
- net TX2: now also J25.2
- net TX_TELEM renamed TX1
- net TX1: now also J24.2
- new net: R20.2, R21.1, U9.5 (ADJ)
- new net VBat: C15.1, J23.1 (Pin_1), U9.1 (EN), U9.2 (VIN)
- no-connect marks 31 -> 73
Other:
- note added: "+5V In"
- note added: "Activity LED"
- note added: "BEC"
- note added: "Connectors"
- note added: "GPIO"
- note added: "I2C"
- note added: "LED Indicators"
- note added: "On-board Power"
- note added: "SPI"
- note added: "Settings"
- note added: "UART0"
- note added: "UART1"
- note added: "UART2"
- note removed: "ACtivity LED"
- note removed: "Fan"
- note removed: "Miscellaneous"
- moved on the sheet: C11, C12, C13, C14, D7, D8, R15, R16, R17, R18, R19, U3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

Commit message: pre-check schematic layout
Parts:
- C10: footprint (none) -> Capacitor_SMD:C_0603_1608Metric_Pad1.08x0.95mm_HandSolder
- R1, R10, R11, R17, R18, R19, R20, R21: footprint (none) -> Resistor_SMD:R_0603_1608Metric_Pad0.98x0.95mm_HandSolder
- R12, R13, R14: footprint (none) -> Resistor_SMD:R_0402_1005Metric_Pad0.72x0.64mm_HandSolder
Changed lines of the file:
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@@
 			)
 		)
-		(property "Footprint" ""
+		(property "Footprint" "Resistor_SMD:R_0603_1608Metric_Pad0.98x0.95mm_HandSolder"
 			(at 521.97 83.82 0)
 			(effects
@@
 			)
 		)
-		(property "Footprint" ""
+		(property "Footprint" "Resistor_SMD:R_0603_1608Metric_Pad0.98x0.95mm_HandSolder"
 			(at 68.58 262.89 0)
 			(effects
@@
 			)
 		)
-		(property "Footprint" ""
+		(property "Footprint" "Resistor_SMD:R_0603_1608Metric_Pad0.98x0.95mm_HandSolder"
 			(at 68.58 270.51 0)
 			(effects
@@
 			)
 		)
-		(property "Footprint" ""
+		(property "Footprint" "Capacitor_SMD:C_0603_1608Metric_Pad1.08x0.95mm_HandSolder"
 			(at 523.24 46.99 0)
 			(effects
@@
 			)
 		)
-		(property "Footprint" ""
+		(property "Footprint" "Resistor_SMD:R_0603_1608Metric_Pad0.98x0.95mm_HandSolder"
 			(at 305.435 205.105 0)
 			(effects
@@
 			)
 		)
-		(property "Footprint" ""
+		(property "Footprint" "Resistor_SMD:R_0402_1005Metric_Pad0.72x0.64mm_HandSolder"
 			(at 472.44 153.035 0)
 			(effects
@@
 			)
 		)
-		(property "Footprint" ""
+		(property "Footprint" "Resistor_SMD:R_0603_1608Metric_Pad0.98x0.95mm_HandSolder"
 			(at 521.97 78.74 0)
 			(effects
@@
 			)
 		)
-		(property "Footprint" ""
+		(property "Footprint" "Resistor_SMD:R_0402_1005Metric_Pad0.72x0.64mm_HandSolder"
 			(at 467.995 153.035 0)
 			(effects
@@
 			)
 		)
-		(property "Footprint" ""
+		(property "Footprint" "Resistor_SMD:R_0402_1005Metric_Pad0.72x0.64mm_HandSolder"
 			(at 539.75 152.4 0)
 			(effects
@@
 			)
 		)
-		(property "Footprint" ""
+		(property "Footprint" "Resistor_SMD:R_0603_1608Metric_Pad0.98x0.95mm_HandSolder"
 			(at 198.12 273.685 0)
 			(effects
@@
 			)
 		)
-		(property "Footprint" ""
+		(property "Footprint" "Resistor_SMD:R_0603_1608Metric_Pad0.98x0.95mm_HandSolder"
 			(at 67.945 197.485 0)
 			(effects
@@
 			)
 		)
-		(property "Footprint" ""
+		(property "Footprint" "Resistor_SMD:R_0603_1608Metric_Pad0.98x0.95mm_HandSolder"
 			(at 137.795 279.4 0)
 			(effects

Commit message: added PCIe to PCBA
Parts:
- removed J12, J15, J20, J21: Conn_01x01, symbol Connector_Generic:Conn_01x01
- removed J3: THD-02-R, symbol Connector_Generic:Conn_02x02_Odd_Even
- removed J6, J9: Conn_01x01, TestPoint:TestPoint_THTPad_3.0x3.0mm_Drill1.5mm, symbol Connector_Generic:Conn_01x01
- removed Module2: ComputeModule5-CM5, CM5IO:Raspberry-Pi-5-Compute-Module, symbol CM5IO:ComputeModule5-CM5
- removed U9: MIC29752WT, Package_TO_SOT_THT:TO-247-5_Vertical, symbol Regulator_Linear:MIC29752WT
- added C17, C18, C19, C20, C21, C22: 10uF, symbol Device:C_Small
- added C23: 10nF, symbol Device:C_Small
- added D9: LED, LED_SMD:LED_0805_2012Metric_Pad1.15x1.40mm_HandSolder, symbol Device:LED
- added J3: Bus_M.2_Socket_M, CM5IO:M.2 M Key socket, symbol CM5IO:Bus_M.2_Socket_M
- added J6, J9: Conn_02x01, Jumper:SolderJumper-2_P1.3mm_Open_TrianglePad1.0x1.5mm, symbol Connector_Generic:Conn_02x01
- added L1: 2.2uH, symbol Device:L_Small
- added unit 2 of Module1
- added R22: 2.2K | 1%, symbol Device:R_Small
- added R23: 1K, symbol Device:R_Small
- added U10: ASEK-32.768KHZ-L-R-T, Crystal:Crystal_SMD_3225-4Pin_3.2x2.5mm, symbol CM5IO:ASEK-32.768KHZ-L-R-T
- added U9: AP3441SHE-7B, Package_DFN_QFN:DFN-8-1EP_2x2mm_P0.5mm_EP1.05x1.75mm, symbol CM5IO:AP3441SHE-7B
- C1, C2: footprint (none) -> Capacitor_SMD:C_0402_1005Metric
- C10: value 1uF -> 1nF; footprint Capacitor_SMD:C_0603_1608Metric_Pad1.08x0.95mm_HandSolder -> Capacitor_SMD:C_0402_1005Metric
- C11, C12, C13, C8: footprint (none) -> Capacitor_SMD:C_0805_2012Metric
- C14: footprint (none) -> Capacitor_Tantalum_SMD:CP_EIA-7343-31_Kemet-D
- C15: value 22uF -> 10uF
- C3, C9: footprint Capacitor_SMD:C_0603_1608Metric_Pad1.08x0.95mm_HandSolder -> Capacitor_SMD:C_0805_2012Metric_Pad1.18x1.45mm_HandSolder
- C4, C6: footprint (none) -> Capacitor_SMD:C_0805_2012Metric_Pad1.18x1.45mm_HandSolder
- C5, C7: footprint (none) -> Capacitor_SMD:C_1206_3216Metric_Pad1.33x1.80mm_HandSolder
- D1, D2, D3, D4, D5, D6: footprint LED_SMD:LED_0603_1608Metric_Pad1.05x0.95mm_HandSolder -> LED_SMD:LED_0805_2012Metric_Pad1.15x1.40mm_HandSolder
- D7, D8: footprint (none) -> LED_SMD:LED_0603_1608Metric
- J10: footprint TestPoint:TestPoint_Loop_D2.54mm_Drill1.5mm_Beaded -> TestPoint:TestPoint_Pad_1.0x1.0mm
- J11, J13, J14, J16, J17, J18, J19: footprint (none) -> TestPoint:TestPoint_Pad_1.0x1.0mm
- JP1, JP2, JP3, JP4, JP5, JP6: footprint (none) -> Jumper:SolderJumper-2_P1.3mm_Open_Pad1.0x1.5mm
- JP7, JP8: footprint (none) -> Jumper:SolderJumper-2_P1.3mm_Open_RoundedPad1.0x1.5mm
- R1, R10, R11, R17, R18, R19: footprint Resistor_SMD:R_0603_1608Metric_Pad0.98x0.95mm_HandSolder -> Resistor_SMD:R_0402_1005Metric
- R12, R13, R14: footprint Resistor_SMD:R_0402_1005Metric_Pad0.72x0.64mm_HandSolder -> Resistor_SMD:R_0402_1005Metric
- R15, R16, R4, R5: footprint (none) -> Resistor_SMD:R_0805_2012Metric_Pad1.20x1.40mm_HandSolder
- R2, R3, R6, R7, R8, R9: footprint Resistor_SMD:R_0603_1608Metric_Pad0.98x0.95mm_HandSolder -> Resistor_SMD:R_0805_2012Metric_Pad1.20x1.40mm_HandSolder
- R20: value 420R -> 100K; footprint Resistor_SMD:R_0603_1608Metric_Pad0.98x0.95mm_HandSolder -> (none)
- R21: value 140R -> 10K | 1%; footprint Resistor_SMD:R_0603_1608Metric_Pad0.98x0.95mm_HandSolder -> (none)
- TP1, TP2, TP3, TP4, TP5, TP6: footprint (none) -> TestPoint:TestPoint_Pad_D1.0mm
Connections:
- net VBat is gone; now on net +5v: C15.1, J23.1 (Pin_1)
- net +5v: now also C17.1, U9.3 (VIN); no longer R20.1
- net DPHY0_D0_N: now also Module1.115 (MIPI0_D0_N)
- net DPHY0_D0_P: now also Module1.117 (MIPI0_D0_P)
- net DPHY0_D1_N: now also Module1.121 (MIPI0_D1_N)
- net DPHY0_D1_P: now also Module1.123 (MIPI0_D1_P)
- net DPHY0_D2_N: now also Module1.133 (MIPI0_D2_N)
- net DPHY0_D2_P: now also Module1.135 (MIPI0_D2_P)
- net DPHY0_D3_N: now also Module1.139 (MIPI0_D3_N)
- net DPHY0_D3_P: now also Module1.141 (MIPI0_D3_P)
- net DPHY1_C_N: now also Module1.187 (MIPI1_C_N)
- net DPHY1_C_P: now also Module1.189 (MIPI1_C_P)
- net DPHY1_D0_N: now also Module1.175 (MIPI1_D0_N)
- net DPHY1_D0_P: now also Module1.177 (MIPI1_D0_P)
- net DPHY1_D1_N: now also Module1.181 (MIPI1_D1_N)
- net DPHY1_D1_P: now also Module1.183 (MIPI1_D1_P)
- net DPHY1_D2_N: now also Module1.193 (MIPI1_D2_N)
- net DPHY1_D2_P: now also Module1.195 (MIPI1_D2_P)
- net DPHY1_D3_N: now also Module1.194 (MIPI1_D3_N)
- net DPHY1_D3_P: now also Module1.196 (MIPI1_D3_P)
- net DPHY_C_N: now also Module1.127 (MIPI0_C_N)
- net DPHY_C_P: now also Module1.129 (MIPI0_C_P)
- net GND: now also R20.2, C17.2, C19.2, C20.2, C21.2, C22.2, C23.2, J3.1 (GND), J3.15 (GND), J3.21 (GND), J3.27 (GND), J3.3 (GND), J3.33 (GND), J3.39 (GND), J3.45 (GND), J3.51 (GND), J3.57 (GND), J3.71 (GND), J3.73 (GND), J3.75 (GND), J3.9 (GND), J3.M1 (GND2230), J3.M2 (GND2242), J3.M3 (GND2260), J3.M4 (GND2280), J3.S1, J3.S2, Module1.107 (GND), Module1.108 (GND), Module1.113 (GND), Module1.114 (GND), Module1.119 (GND), Module1.120 (GND), Module1.125 (GND), Module1.126 (GND), Module1.131 (GND), Module1.132 (GND), Module1.137 (GND), Module1.138 (GND), Module1.144 (GND), Module1.150 (GND), Module1.155 (GND), Module1.156 (GND), Module1.161 (GND), Module1.162 (GND), Module1.167 (GND), Module1.168 (GND), Module1.173 (GND), Module1.174 (GND), Module1.179 (GND), Module1.180 (GND), Module1.185 (GND), Module1.186 (GND), Module1.191 (GND), Module1.192 (GND), Module1.197 (GND), Module1.198 (GND), R22.2, U10.2 (GND), U9.4 (PGND), U9.8 (SGND), U9.9 (PAD); no longer R21.2
- net TR0_TAP: now also J9.1 (Pin_1)
- net TR1_TAP: now also J6.1 (Pin_1)
- net TR2_TAP: now also J6.2 (Pin_2)
- net TR3_TAP: now also J9.2 (Pin_2)
- net USB2_N: now also Module1.103 (USB2_N)
- net USB2_P: now also Module1.105 (USB2_P)
- net USB3-0-D_N: now also Module1.136 (USB3-0-D_N)
- net USB3-0-D_P: now also Module1.134 (USB3-0-D_P)
- net USB3-1-D_N: now also Module1.165 (USB3-1-D_N)
- net USB3-1-D_P: now also Module1.163 (USB3-1-D_P)
- net USBOTG: now also Module1.101 (USB_OTG_ID)
- net VBUS_EN: now also Module1.111 (VBUS_EN)
- net at C7.1, R6.2, R7.2: now also C6.2
- net M2_3v3: now reaches R21.1
- net M2_3v3: now also C18.1, C19.1, C20.1, C21.1, C22.1, C23.1, D9.2 (A), J3.12 (3.3V), J3.14 (3.3V), J3.16 (3.3V), J3.18 (3.3V), J3.2 (3.3V), J3.4 (3.3V), J3.70 (3.3V), J3.72 (3.3V), J3.74 (3.3V), L1.2, U10.1 (EN), U10.4 (VDD); no longer R20.2
- net at C5.1, R4.2, R5.2: now also C4.2
- new net: J3.10 (DAS/~{DSS}/~{LED1}), R23.2
- new net: J3.68 (SUSCLK), U10.3 (Out)
- new net: D9.1 (K), R23.1
- new net: L1.1, U9.6 (LX)
- new net FB: C18.2, R21.2, R22.1, U9.1 (FB)
- new net PCIE_CLK_N: J3.53 (REFCLKn), Module1.112 (PCIe_CLK_N)
- new net PCIE_CLK_P: J3.55 (REFCLKp), Module1.110 (PCIe_CLK_P)
- new net PCIE_PWR_EN: Module1.106 (PCIE_PWR_EN), R20.1, U9.7 (EN)
- new net PCIE_RX_N: J3.43 (PETp0), Module1.118 (PCIe_RX_N)
- new net PCIE_RX_P: J3.41 (PETn0), Module1.116 (PCIe_RX_P)
- new net PCIE_TX_N: J3.49 (PERp0), Module1.124 (PCIe_TX_N)
- new net PCIE_TX_P: J3.47 (PERn0), Module1.122 (PCIe_TX_P)
- new net PCIE_nCLKREQ: J3.52 (~{CLKREQ}), Module1.102 (PCIe_nCLKREQ)
- new net PCIE_nRST: J3.50 (~{PERST}), Module1.109 (PCIe_nRST)
- new net PCIE_nWAKE: J3.54 (~{PEWAKE}), Module1.104 (PCIE_nWAKE)
- no-connect marks 73 -> 78
Other:
- note added: "PCIe"
- note added: "PCIe Power"
- note removed: "+5V In"
- moved on the sheet: C1, C2, J10, J11, J13, J14, J16, J17, J18, J19, J23, J8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

Commit message: added PCIe slot
Parts:
- removed TP36: TestPoint, TestPoint:TestPoint_Pad_D1.0mm, symbol Connector:TestPoint
- added M1: M.2 Screw, symbol CM5IO:M.2_Screw
- added M2, M3: M.2 Solder Nut, symbol CM5IO:SolderNut
- C10: value 1nF -> 100nF
- C15, C16, C19, C20, C21, C22: footprint (none) -> Capacitor_SMD:C_0805_2012Metric
- C17: value 10uF -> 100nF; footprint (none) -> Capacitor_SMD:C_0402_1005Metric
- C18: value 10uF -> 4.7nF; footprint (none) -> Capacitor_SMD:C_0402_1005Metric
- C23: value 10nF -> 100nF; footprint (none) -> Capacitor_SMD:C_0402_1005Metric
- L1: footprint (none) -> CM5IO:L_Bourns_SRP5030CC
- R17: value 1k -> 1K
- R20: value 100K -> 100K | 1%; footprint (none) -> Resistor_SMD:R_0402_1005Metric
- R21, R22, R23: footprint (none) -> Resistor_SMD:R_0402_1005Metric
Connections:
- net GPIO2: now also JP7.2 (B), R14.2
- net GPIO3: no longer JP8.2 (B), R13.1
- net SCL0: no longer JP7.2 (B), R14.2
- net SDA1: now also JP8.2 (B), R13.1
Other:
- note added: "3.3V logic level"
- note added: "Flight Controller UART"
- note added: "PCIe M2"
- note added: "Power In"
- note added: "Power Out"
- note added: "USB VBUS Current Limit Switch"
- note removed: "BEC"
- note removed: "Current Limit Switch"
- note removed: "PCIe"
- note removed: "Power"
- moved on the sheet: C11, C12, C13, C14, J7, Module1A, Module1B, R18, R20, S1, U8

Commit message: started PCB layout
Parts:
- removed J10, J11, J13, J14, J16, J17, J18, J19: Conn_01x01, TestPoint:TestPoint_Pad_1.0x1.0mm, symbol Connector_Generic:Conn_01x01
- J1: footprint CM5IO:EDAC 690-019-298-412 -> Connector_USB:USB_C_Receptacle_GCT_USB4105-xx-A_16P_TopMnt_Horizontal
Connections:
- net GPIO2: no longer J5.20 (Pin_20), JP7.2 (B), R14.2
- net GPIO3: no longer J4.21 (Pin_21), Module1.82 (SDA0)
- net RX1 renamed RX_TELEM
- net RX2 renamed RX_CRSF
- net TX1 renamed TX_TELEM
- net TX2 renamed TX_CRSF
- new net SCL1: J5.20 (Pin_20), JP7.2 (B), R14.2
- new net SDA0: J4.21 (Pin_21), Module1.82 (SDA0)
Other:
- note removed: "Power Out"
- moved on the sheet: TP10, TP11, TP12, TP13, TP14, TP15, TP16, TP17, TP18, TP19, TP20, TP21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
