File: PCB/specter/specter.kicad_sch (KiCad schematic)
At the start: 132 parts, among them J1 USB_C_Receptacle_USB2.0_16P, J2 Micro_SD_Card_Det2, J22 SM04B-SRSS-TB_LF__SN_, J23 Conn_01x01, J24 SM04B-SRSS-TB_LF__SN_, J25 SM04B-SRSS-TB_LF__SN_, J26 SM04B-SRSS-TB_LF__SN_, J27 SM06B-SRSS-TB_LF__SN_, J28 SM06B-SRSS-TB_LF__SN_, J29 SM06B-SRSS-TB_LF__SN_, J3 Bus_M.2_Socket_M, J30 SM06B-SRSS-TB_LF__SN_, J4 Conn_01x22_Socket, J5 Conn_01x22_Socket, J6 Conn_02x01, J7 Conn_01x03, J8 Conn_01x01, J9 Conn_02x01, M1 M.2 Screw, M2 M.2 Solder Nut, M3 M.2 Solder Nut, U1 FT232RL, U10 ASEK-32.768KHZ-L-R-T, U2 FT232RL, U3 RT9742GGJ5, U4 MagJack-A70-112-331N126, U5 TPD4EUSB30, U6 TPD4EUSB30, U7 74LVC1G07_copy, U8 AP2553W6, U9 AP3441SHE-7B

Commit message: finishing touches
Parts:
- removed TP10, TP11, TP12, TP13, TP14, TP15, TP16, TP17, TP18, TP19, TP20, TP21, TP22, TP23, TP24, TP25, TP26, TP27, TP28, TP29, TP30, TP31, TP32, TP33, TP34, TP7, TP8, TP9: TestPoint, TestPoint:TestPoint_Pad_D1.0mm, symbol Connector:TestPoint
Other:
- note removed: "Test Point Breakout"
- moved on the sheet: C15, C16, C17, C18, C19, C20, C21, C22, L1, R20, R21, R22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

Commit message: final PCB changes
Parts:
- removed C10: 100nF, Capacitor_SMD:C_0402_1005Metric, symbol Device:C_Small
- removed J6, J9: Conn_02x01, Jumper:SolderJumper-2_P1.3mm_Open_TrianglePad1.0x1.5mm, symbol Connector_Generic:Conn_02x01
- removed R10, R11: 470R, Resistor_SMD:R_0402_1005Metric, symbol Device:R_Small
- removed R15, R16: 0R, Resistor_SMD:R_0805_2012Metric_Pad1.20x1.40mm_HandSolder, symbol Device:R_Small
- removed R4, R6: 0, Resistor_SMD:R_0805_2012Metric_Pad1.20x1.40mm_HandSolder, symbol Device:R_Small
- removed U4: MagJack-A70-112-331N126, CM5IO:TRJG0926HENL, symbol CM5IO:MagJack-A70-112-331N126
- removed U5, U6: TPD4EUSB30, Package_SON:USON-10_2.5x1.0mm_P0.5mm, symbol CM5IO:TPD4EUSB30
- added J6, J9: DF40C-100DS-0.4V_51_, DF40C-100DS-0:HIROSE_DF40C-100DS-0.4V_51_, symbol DF40C-100DS-0.4V_51_:DF40C-100DS-0.4V_51_
- Module1: now left out of the parts list
Connections:
- net GPIO_VREF is gone; now on net +3.3v: Module1.78 (GPIO_VREF(1.8v/3.3v_Input)), R13.2, R14.1
- net VBUS: now also C4.2, C5.1, C6.2, C7.1, R5.2, R7.2
Other:
- note removed: "Ethernet"
- note removed: "PoE"
- moved on the sheet: J4, J5, JP7, JP8, R12, R13, R14
